File: keyboard.kicad_sch (KiCad schematic)
At the start: 79 parts, among them J6 Conn_01x09_Male, SW10 I @, SW11 O ", SW12 P \, SW13 A &, SW14 S /, SW15 D 4, SW16 F 5, SW17 G 6, SW18 H $, SW19 J !, SW20 K ;, SW21 L ', SW22 Del, SW23 { }, SW24 Z %, SW25 X 7, SW26 C 8, SW27 V 9, SW28 B #, SW29 N ?, SW3 Q |, SW30 M :, SW31 [ ], SW32 Enter, SW33 Shift, SW34 + -, SW35 0 ~, SW36 Tab ^, SW37 Space, SW38 , ., SW39 < >, SW4 W *, SW40 Cap, SW5 E 1, SW6 R 2, SW7 T 3, SW8 Y (, SW9 U )

Commit message: update silkscreen to replace 'tab' with '='
Parts:
- SW36: value Tab ^ -> = ^
Changed lines of the file:
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@@
     (in_bom yes) (on_board yes)
     (property "Reference" "SW36" (id 0) (at 139.7 138.811 0))
-    (property "Value" "Tab ^" (id 1) (at 139.7 141.1224 0))
+    (property "Value" "= ^" (id 1) (at 139.7 141.1224 0))
     (property "Footprint" "e-tinkers:SW_PUSH_6mm_XKB_TC-1102-X-X-X" (id 2) (at 139.7 140.97 0)
       (effects (font (size 1.27 1.27)) hide)
